File: inv_pendulum.brd (EAGLE design)
At the start: 49.2 x 74.9 mm, 9 parts

Commit message: update design
Parts:
- U$5, U$6: value TBLOCK-2 -> (none); device akizuki_MOSFET:TBLOCK-2 -> SparkFun-Connectors:1X02_LOCK_LONGPADS
- moved U$1 11.4 mm to (44.5, 49.5)
- moved U$3 8.89 mm to (27.9, 49.5)
- moved U$5 6.48 mm to (45.7, 25.4)
- moved U$6 6.48 mm to (45.7, 7.62)
- moved POWER 6.48 mm to (40.6, 68.6)
- moved R1 2.84 mm to (24.1, 68.6)
- moved R2 2.84 mm to (11.4, 68.6)
- moved U$2 2.54 mm to (24.1, 16.5)
- moved U$4 2.54 mm to (11.4, 49.5)
Routing:
- net N$5: track 110.1 -> 61.0 mm, vias 2 -> 0
- net 3V3: track 137.6 -> 180.6 mm, vias 2 -> 0
- net N$4: track 25.8 -> 68.8 mm
- net IN1: track 44.6 -> 84.8 mm, vias 0 -> 2
- net PWM1: track 71.3 -> 34.0 mm
- net GND: track 175.9 -> 143.2 mm, vias 0 -> 4
- net N$11: track 87.4 -> 115.9 mm
- net N$10: track 105.7 -> 80.7 mm
- net 6V: track 124.4 -> 136.3 mm, vias 6 -> 2
- net SCL: track 94.0 -> 101.9 mm, vias 5 -> 2
- net SDA: track 116.8 -> 123.3 mm
- net IN2: track 44.1 -> 49.0 mm, vias 0 -> 2
Other:
- board size 49.2 x 74.9 mm -> 55.5 x 77.5 mm

Commit message: update design
Routing:
- net N$10: track 80.7 -> 86.4 mm
- net 6V: track 136.3 -> 138.4 mm
Changed lines of the file:
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@@
 <via x="15.24" y="10.16" extent="1-16" drill="0.7" diameter="1.4224"/>
 <wire x1="15.24" y1="10.16" x2="16.51" y2="11.43" width="0.762" layer="1"/>
-<wire x1="16.51" y1="11.43" x2="17.78" y2="17.78" width="0.762" layer="1"/>
-<wire x1="17.78" y1="17.78" x2="15.24" y2="19.05" width="0.762" layer="1"/>
-<wire x1="15.24" y1="19.05" x2="13.97" y2="22.86" width="0.762" layer="1"/>
-<wire x1="13.97" y1="22.86" x2="13.97" y2="26.67" width="0.762" layer="1"/>
-<wire x1="13.97" y1="26.67" x2="12.7" y2="26.67" width="0.762" layer="1"/>
-<wire x1="12.7" y1="26.67" x2="11.43" y2="29.21" width="0.762" layer="1"/>
-<wire x1="11.43" y1="29.21" x2="6.35" y2="31.75" width="0.762" layer="1"/>
-<wire x1="6.35" y1="31.75" x2="5.08" y2="31.75" width="0.762" layer="1"/>
-<wire x1="5.08" y1="31.75" x2="5.08" y2="54.61" width="0.762" layer="1"/>
+<wire x1="16.51" y1="11.43" x2="16.51" y2="17.78" width="0.762" layer="1"/>
+<wire x1="16.51" y1="17.78" x2="13.97" y2="17.78" width="0.762" layer="1"/>
+<wire x1="13.97" y1="17.78" x2="13.97" y2="26.67" width="0.762" layer="1"/>
+<wire x1="13.97" y1="26.67" x2="11.43" y2="29.21" width="0.762" layer="1"/>
+<wire x1="11.43" y1="29.21" x2="5.08" y2="29.21" width="0.762" layer="1"/>
+<wire x1="5.08" y1="29.21" x2="5.08" y2="54.61" width="0.762" layer="1"/>
 <via x="5.08" y="54.61" extent="1-16" drill="0.7" diameter="1.4224"/>
 <wire x1="5.08" y1="54.61" x2="7.62" y2="55.88" width="0.762" layer="16"/>
@@
 <wire x1="20.32" y1="2.54" x2="20.32" y2="10.16" width="0.762" layer="16"/>
 <via x="20.32" y="10.16" extent="1-16" drill="0.7" diameter="1.4224"/>
-<wire x1="20.32" y1="10.16" x2="21.59" y2="12.7" width="0.762" layer="1"/>
-<wire x1="21.59" y1="12.7" x2="20.32" y2="19.05" width="0.762" layer="1"/>
-<wire x1="20.32" y1="19.05" x2="16.51" y2="25.4" width="0.762" layer="1"/>
-<wire x1="16.51" y1="25.4" x2="12.7" y2="30.48" width="0.762" layer="1"/>
-<wire x1="12.7" y1="30.48" x2="10.16" y2="31.75" width="0.762" layer="1"/>
-<wire x1="10.16" y1="31.75" x2="6.35" y2="35.56" width="0.762" layer="1"/>
-<wire x1="6.35" y1="35.56" x2="6.35" y2="41.91" width="0.762" layer="1"/>
+<wire x1="20.32" y1="10.16" x2="19.05" y2="12.7" width="0.762" layer="1"/>
+<wire x1="19.05" y1="12.7" x2="19.05" y2="19.05" width="0.762" layer="1"/>
+<wire x1="19.05" y1="19.05" x2="15.24" y2="19.05" width="0.762" layer="1"/>
+<wire x1="15.24" y1="19.05" x2="15.24" y2="27.94" width="0.762" layer="1"/>
+<wire x1="15.24" y1="27.94" x2="12.7" y2="30.48" width="0.762" layer="1"/>
+<wire x1="12.7" y1="30.48" x2="6.35" y2="30.48" width="0.762" layer="1"/>
+<wire x1="6.35" y1="30.48" x2="6.35" y2="41.91" width="0.762" layer="1"/>
 <wire x1="6.35" y1="41.91" x2="8.89" y2="43.18" width="0.762" layer="1"/>
 <via x="8.89" y="43.18" extent="1-16" drill="0.7" diameter="1.4224"/>

Commit message: update design
Routing:
- net N$10: track 86.4 -> 85.6 mm
- net 6V: track 138.4 -> 137.6 mm
Changed lines of the file:
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@@
 <wire x1="16.51" y1="17.78" x2="13.97" y2="17.78" width="0.762" layer="1"/>
 <wire x1="13.97" y1="17.78" x2="13.97" y2="26.67" width="0.762" layer="1"/>
-<wire x1="13.97" y1="26.67" x2="11.43" y2="29.21" width="0.762" layer="1"/>
-<wire x1="11.43" y1="29.21" x2="5.08" y2="29.21" width="0.762" layer="1"/>
-<wire x1="5.08" y1="29.21" x2="5.08" y2="54.61" width="0.762" layer="1"/>
+<wire x1="13.97" y1="26.67" x2="10.16" y2="30.48" width="0.762" layer="1"/>
+<wire x1="10.16" y1="30.48" x2="5.08" y2="30.48" width="0.762" layer="1"/>
+<wire x1="5.08" y1="30.48" x2="5.08" y2="54.61" width="0.762" layer="1"/>
 <via x="5.08" y="54.61" extent="1-16" drill="0.7" diameter="1.4224"/>
 <wire x1="5.08" y1="54.61" x2="7.62" y2="55.88" width="0.762" layer="16"/>
@@
 <wire x1="19.05" y1="19.05" x2="15.24" y2="19.05" width="0.762" layer="1"/>
 <wire x1="15.24" y1="19.05" x2="15.24" y2="27.94" width="0.762" layer="1"/>
-<wire x1="15.24" y1="27.94" x2="12.7" y2="30.48" width="0.762" layer="1"/>
-<wire x1="12.7" y1="30.48" x2="6.35" y2="30.48" width="0.762" layer="1"/>
-<wire x1="6.35" y1="30.48" x2="6.35" y2="41.91" width="0.762" layer="1"/>
+<wire x1="15.24" y1="27.94" x2="11.43" y2="31.75" width="0.762" layer="1"/>
+<wire x1="11.43" y1="31.75" x2="6.35" y2="31.75" width="0.762" layer="1"/>
+<wire x1="6.35" y1="31.75" x2="6.35" y2="41.91" width="0.762" layer="1"/>
 <wire x1="6.35" y1="41.91" x2="8.89" y2="43.18" width="0.762" layer="1"/>
 <via x="8.89" y="43.18" extent="1-16" drill="0.7" diameter="1.4224"/>
